File: KiCad/CodyKeyboard/CodyKeyboard.kicad_sch (KiCad schematic)
At the start: 32 parts, among them SW1 "CODY", SW10 "B", SW11 "N", SW12 "M", SW13 "L", SW14 "K", SW15 "J", SW16 "H", SW17 "G", SW18 "F", SW19 "D", SW2 "META", SW20 "S", SW21 "A", SW22 "Q", SW23 "W", SW24 "E", SW25 "R", SW26 "T", SW27 "Y", SW28 "U", SW29 "I", SW3 "ARROW", SW30 "O", SW31 "P", SW4 "SPACE1", SW5 "SPACE2", SW6 "Z", SW7 "X", SW8 "C", SW9 "V"

Commit message: Add exported PDF schematics
Parts:
- J1: value (none) -> Keyboard Connector
Changed lines of the file:
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@@
       (effects (font (size 1.27 1.27)) (justify right))
     )
-    (property "Value" "" (id 1) (at 221.6912 100.7618 0)
+    (property "Value" "Keyboard Connector" (id 1) (at 221.6912 100.7618 0)
       (effects (font (size 1.27 1.27)) (justify right))
     )
