File: KiCad/CodyComputer/CPU.kicad_sch (KiCad schematic)
At the start: 5 parts, among them U5 W65C02SxP, U6 AS6C1008

Commit message: Add debug power connector to schematic
Parts:
- U5: footprint Package_DIP:DIP-40_W15.24mm_Socket -> Package_DIP:DIP-40_W15.24mm_Socket_LongPads
- U6: footprint Package_DIP:DIP-32_W15.24mm_Socket -> Package_DIP:DIP-32_W15.24mm_Socket_LongPads
Changed lines of the file:
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@@
   (title_block
     (title "65C02 Microprocessor and Static RAM")
-    (date "2023-04-18")
-    (rev "A")
+    (date "2025-01-06")
+    (rev "B")
   )
   (junction (at 38.1 88.9) (diameter 0) (color 0 0 0 0)
@@
     (property "Reference" "U5" (id 0) (at 86.36 57.15 0))
     (property "Value" "W65C02SxP" (id 1) (at 86.36 59.69 0))
-    (property "Footprint" "Package_DIP:DIP-40_W15.24mm_Socket" (id 2) (at 78.74 45.72 0)
+    (property "Footprint" "Package_DIP:DIP-40_W15.24mm_Socket_LongPads" (id 2) (at 78.74 45.72 0)
       (effects (font (size 1.27 1.27)) hide)
     )
@@
     (property "Reference" "U6" (id 0) (at 210.82 69.85 0))
     (property "Value" "AS6C1008" (id 1) (at 210.82 72.39 0))
-    (property "Footprint" "Package_DIP:DIP-32_W15.24mm_Socket" (id 2) (at 203.2 97.79 0)
-      (effects (font (size 1.27 1.27)) hide)
-    )
+    (property "Footprint" "Package_DIP:DIP-32_W15.24mm_Socket_LongPads" (id 2) (at 203.2 97.79 0)
+      (effects (font (size 1.27 1.27)) hide)
+    )
