File: KiCad/CodyComputer/IO.kicad_sch (KiCad schematic)
At the start: 24 parts, among them J6 Cody Expansion/Cartridge Port, J7 Keyboard Connector, U7 W65C22SxP, U8 4051

Commit message: Add exported PDF schematics
Parts:
- J8: value (none) -> Joystick 1
- J9: value (none) -> Joystick 2
Changed lines of the file:
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@@
       (effects (font (size 1.27 1.27)) (justify left))
     )
-    (property "Value" "" (id 1) (at 207.772 154.813 0)
+    (property "Value" "Joystick 2" (id 1) (at 207.772 154.813 0)
       (effects (font (size 1.27 1.27)) (justify left))
     )
@@
       (effects (font (size 1.27 1.27)) (justify left))
     )
-    (property "Value" "" (id 1) (at 207.772 106.553 0)
-      (effects (font (size 1.27 1.27)) (justify left))
-    )
+    (property "Value" "Joystick 1" (id 1) (at 207.772 106.553 0)
+      (effects (font (size 1.27 1.27)) (justify left))
+    )

Commit message: Add debug power connector to schematic
Parts:
- U7: footprint Package_DIP:DIP-40_W15.24mm_Socket -> Package_DIP:DIP-40_W15.24mm_Socket_LongPads
- U8: footprint Package_DIP:DIP-16_W7.62mm_Socket -> Package_DIP:DIP-16_W7.62mm_Socket_LongPads
Changed lines of the file:
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@@
   (title_block
     (title "65C22 VIA, Keyboard/Joystick, Cartridge, SPI")
-    (date "2023-04-18")
-    (rev "A")
+    (date "2025-01-06")
+    (rev "B")
   )
   (junction (at 153.67 66.04) (diameter 0) (color 0 0 0 0)
@@
     (property "Reference" "U7" (id 0) (at 77.47 44.45 0))
     (property "Value" "W65C22SxP" (id 1) (at 77.47 46.99 0))
-    (property "Footprint" "Package_DIP:DIP-40_W15.24mm_Socket" (id 2) (at 69.85 77.47 0)
+    (property "Footprint" "Package_DIP:DIP-40_W15.24mm_Socket_LongPads" (id 2) (at 69.85 77.47 0)
       (effects (font (size 1.27 1.27)) hide)
     )
@@
       (effects (font (size 1.27 1.27)) (justify left))
     )
-    (property "Footprint" "Package_DIP:DIP-16_W7.62mm_Socket" (id 2) (at 232.41 55.88 0)
-      (effects (font (size 1.27 1.27)) hide)
-    )
+    (property "Footprint" "Package_DIP:DIP-16_W7.62mm_Socket_LongPads" (id 2) (at 232.41 55.88 0)
+      (effects (font (size 1.27 1.27)) hide)
+    )
